Commit message: add urdf files of workcell and eef

File: aubo_robot/aubo_description/urdf/aubo_i5.urdf.xacro (robot description, xacro)
@@ -619,10 +619,28 @@
      <collision>
        <geometry>
-          <box size="0.01 0.01 0.01"/>
+          <!--box size="0.01 0.01 0.01"/-->
+        <mesh
+          filename="package://aubo_description/meshes/End-effector.dae" />
        </geometry>
+       <!--origin
+          rpy="0 0 0"
+          xyz="0 0 0.05"/-->
        <origin
           rpy="0 0 0"
           xyz="0 0 0.05"/>
      </collision>
+     <visual>
+       <geometry>
+          <!--box size="0.01 0.01 0.01"/-->
+        <mesh
+          filename="package://aubo_description/meshes/End-effector.dae" />
+       </geometry>
+       <!--origin
+          rpy="0 0 0"
+          xyz="0 0 0.05"/-->
+       <origin
+          rpy="0 0 2.35"
+          xyz="0.089 0.043 -0.04"/>
+     </visual>
   </link>
   <joint

File: aubo_robot/aubo_description/urdf/aubo_i5_robot.urdf.xacro (robot description, xacro)
@@ -30,3 +30,28 @@
     <origin xyz="0.0 0.0 -0.40" rpy="0.0 0.0 0.785" />
   </joint>
+<!-- Workcell -->
+  <link
+    name="workcell">
+    <visual>
+      <origin
+        xyz="-0.39 0.39 -1.15"
+        rpy="0 0 -0.785" />
+      <geometry>
+        <mesh filename="package://aubo_description/meshes/workcell.dae" />
+      </geometry>
+    </visual>
+    <collision>
+      <origin
+        xyz="-0.39 0.39 -1.15"
+        rpy="0 0 -0.785" />
+      <geometry>
+        <mesh filename="package://aubo_description/meshes/workcell.dae" />
+      </geometry>
+    </collision>
+  </link>
+  <joint name="base_to_workcell" type="fixed">
+    <parent link="base_Link"/>
+    <child link="workcell"/>
+  </joint>
+<!-- -->
 </robot>

File: aubo_robot/aubo_description/urdf/aubo_i5_robot_gazebo.urdf.xacro (robot description, xacro)
@@ -28,5 +28,30 @@
     <parent link="base_Link"/>
     <child link="pedestal_Link"/>
-    <origin xyz="0.0 0.0 -0.40" rpy="0.0 0.0 0.0" />
+    <origin xyz="0.0 0.0 -0.40" rpy="0.0 0.0 0.785" />
   </joint>
+<!-- Workcell -->
+  <link
+    name="workcell">
+    <visual>
+      <origin
+        xyz="-0.39 0.39 -1.15"
+        rpy="0 0 -0.785" />
+      <geometry>
+        <mesh filename="package://aubo_description/meshes/workcell.dae" />
+      </geometry>
+    </visual>
+    <collision>
+      <origin
+        xyz="-0.39 0.39 -1.15"
+        rpy="0 0 -0.785" />
+      <geometry>
+        <mesh filename="package://aubo_description/meshes/workcell.dae" />
+      </geometry>
+    </collision>
+  </link>
+  <joint name="base_to_workcell" type="fixed">
+    <parent link="base_Link"/>
+    <child link="workcell"/>
+  </joint>
+<!-- -->
 </robot>

Commit message: added an cross-platform interface to operate the demo

File: aubo_robot/aubo_description/urdf/aubo_i5.urdf.xacro (robot description, xacro)
@@ -634,5 +634,5 @@
           <!--box size="0.01 0.01 0.01"/-->
         <mesh
-          filename="package://aubo_description/meshes/End-effector.dae" />
+          filename="package://aubo_description/meshes/End-effector.STL" />
        </geometry>
        <!--origin

File: aubo_robot/aubo_description/urdf/aubo_i5_robot.urdf.xacro (robot description, xacro)
@@ -38,5 +38,5 @@
         rpy="0 0 -0.785" />
       <geometry>
-        <mesh filename="package://aubo_description/meshes/workcell.dae" />
+        <mesh filename="package://aubo_description/meshes/workcell.STL" />
       </geometry>
     </visual>
